Commit message: Edit urdf mesh path.

File: resources/robots/solo/urdf/solo.urdf (robot description, URDF)
Before this commit: robot solo, 13 links, 12 joints
Links:
- link FL_FOOT: geometry collision mesh filename=../meshes/obj/with_foot/solo_foot.obj; visual mesh filename=../meshes/obj/with_foot/solo_foot.obj
- link FL_LOWER_LEG: geometry collision mesh filename=../meshes/obj/with_foot/solo_lower_leg_left_side.obj; visual mesh filename=../meshes/obj/with_foot/solo_lower_leg_left_side.obj
- link FL_UPPER_LEG: geometry collision mesh filename=../meshes/obj/with_foot/solo_upper_leg_left_side.obj; visual mesh filename=../meshes/obj/with_foot/solo_upper_leg_left_side.obj
- link FR_FOOT: geometry collision mesh filename=../meshes/obj/with_foot/solo_foot.obj; visual mesh filename=../meshes/obj/with_foot/solo_foot.obj
- link FR_LOWER_LEG: geometry collision mesh filename=../meshes/obj/with_foot/solo_lower_leg_right_side.obj; visual mesh filename=../meshes/obj/with_foot/solo_lower_leg_right_side.obj
- link FR_UPPER_LEG: geometry collision mesh filename=../meshes/obj/with_foot/solo_upper_leg_right_side.obj; visual mesh filename=../meshes/obj/with_foot/solo_upper_leg_right_side.obj
- link HL_FOOT: geometry collision mesh filename=../meshes/obj/with_foot/solo_foot.obj; visual mesh filename=../meshes/obj/with_foot/solo_foot.obj
- link HL_LOWER_LEG: geometry collision mesh filename=../meshes/obj/with_foot/solo_lower_leg_left_side.obj; visual mesh filename=../meshes/obj/with_foot/solo_lower_leg_left_side.obj
- link HL_UPPER_LEG: geometry collision mesh filename=../meshes/obj/with_foot/solo_upper_leg_left_side.obj; visual mesh filename=../meshes/obj/with_foot/solo_upper_leg_left_side.obj
- link HR_FOOT: geometry collision mesh filename=../meshes/obj/with_foot/solo_foot.obj; visual mesh filename=../meshes/obj/with_foot/solo_foot.obj
- link HR_LOWER_LEG: geometry collision mesh filename=../meshes/obj/with_foot/solo_lower_leg_right_side.obj; visual mesh filename=../meshes/obj/with_foot/solo_lower_leg_right_side.obj
- link HR_UPPER_LEG: geometry collision mesh filename=../meshes/obj/with_foot/solo_upper_leg_right_side.obj; visual mesh filename=../meshes/obj/with_foot/solo_upper_leg_right_side.obj
- link base_link: geometry collision mesh filename=../meshes/obj/with_foot/solo_body.obj; visual mesh filename=../meshes/obj/with_foot/solo_body.obj

File: resources/robots/solo/urdf/solo12.urdf (robot description, URDF)
Before this commit: robot solo, 17 links, 16 joints
Links:
- link FL_FOOT: geometry collision mesh filename=../meshes/stl/with_foot/solo_foot.stl; visual mesh filename=../meshes/stl/with_foot/solo_foot.stl
- link FL_LOWER_LEG: geometry collision mesh filename=../meshes/stl/with_foot/solo_lower_leg_left_side.stl; visual mesh filename=../meshes/stl/with_foot/solo_lower_leg_left_side.stl
- link FL_SHOULDER: geometry collision mesh filename=../meshes/stl/solo12/solo12_hip_fe_fl.stl; visual mesh filename=../meshes/stl/solo12/solo12_hip_fe_fl.stl
- link FL_UPPER_LEG: geometry collision mesh filename=../meshes/stl/with_foot/solo_upper_leg_left_side.stl; visual mesh filename=../meshes/stl/with_foot/solo_upper_leg_left_side.stl
- link FR_FOOT: geometry collision mesh filename=../meshes/stl/with_foot/solo_foot.stl; visual mesh filename=../meshes/stl/with_foot/solo_foot.stl
- link FR_LOWER_LEG: geometry collision mesh filename=../meshes/stl/with_foot/solo_lower_leg_right_side.stl; visual mesh filename=../meshes/stl/with_foot/solo_lower_leg_right_side.stl
- link FR_SHOULDER: geometry collision mesh filename=../meshes/stl/solo12/solo12_hip_fe_fr.stl; visual mesh filename=../meshes/stl/solo12/solo12_hip_fe_fr.stl
- link FR_UPPER_LEG: geometry collision mesh filename=../meshes/stl/with_foot/solo_upper_leg_right_side.stl; visual mesh filename=../meshes/stl/with_foot/solo_upper_leg_right_side.stl
- link HL_FOOT: geometry collision mesh filename=../meshes/stl/with_foot/solo_foot.stl; visual mesh filename=../meshes/stl/with_foot/solo_foot.stl
- link HL_LOWER_LEG: geometry collision mesh filename=../meshes/stl/with_foot/solo_lower_leg_left_side.stl; visual mesh filename=../meshes/stl/with_foot/solo_lower_leg_left_side.stl
- link HL_SHOULDER: geometry collision mesh filename=../meshes/stl/solo12/solo12_hip_fe_hl.stl; visual mesh filename=../meshes/stl/solo12/solo12_hip_fe_hl.stl
- link HL_UPPER_LEG: geometry collision mesh filename=../meshes/stl/with_foot/solo_upper_leg_left_side.stl; visual mesh filename=../meshes/stl/with_foot/solo_upper_leg_left_side.stl
- link HR_FOOT: geometry collision mesh filename=../meshes/stl/with_foot/solo_foot.stl; visual mesh filename=../meshes/stl/with_foot/solo_foot.stl
- link HR_LOWER_LEG: geometry collision mesh filename=../meshes/stl/with_foot/solo_lower_leg_right_side.stl; visual mesh filename=../meshes/stl/with_foot/solo_lower_leg_right_side.stl
- link HR_SHOULDER: geometry collision mesh filename=../meshes/stl/solo12/solo12_hip_fe_hr.stl; visual mesh filename=../meshes/stl/solo12/solo12_hip_fe_hr.stl
- link HR_UPPER_LEG: geometry collision mesh filename=../meshes/stl/with_foot/solo_upper_leg_right_side.stl; visual mesh filename=../meshes/stl/with_foot/solo_upper_leg_right_side.stl
- link base_link: geometry collision mesh filename=../meshes/stl/solo12/solo_12_base.stl; visual mesh filename=../meshes/stl/solo12/solo_12_base.stl
